Commit message: First draft of depth sensing camera

File: model/camera_bot.gazebo.xacro (robot description, xacro)
@@ -1,56 +1,101 @@
 <?xml version="1.0"?>
 <robot xmlns:xacro="http://www.ros.org/wiki/xacro" name="camera_bot">
-  <!--<gazebo>
-    <plugin name="gazebo_ros_control" filename="libgazebo_ros_control.so">
-      <robotNamespace>camera_bot</robotNamespace>
-      <robotSimType>gazebo_ros_control/DefaultRobotHWSim</robotSimType>
-    </plugin>
-  </gazebo> -->
-  <!-- Base Link -->
-  <gazebo reference="base_link">
-    <material>Gazebo/Green</material>
-  </gazebo>
+	<!--<gazebo>
+		<plugin name="gazebo_ros_control" filename="libgazebo_ros_control.so">
+			<robotNamespace>camera_bot</robotNamespace>
+			<robotSimType>gazebo_ros_control/DefaultRobotHWSim</robotSimType>
+		</plugin>
+	</gazebo> -->
+	<!-- Base Link -->
+	<gazebo reference="base_link">
+		<material>Gazebo/Green</material>
+	</gazebo>
   <!-- camera -->
-  <gazebo reference="camera_link">
-    <material>Gazebo/Red</material>
-    <sensor type="camera" name="camera">
-      <always_on>true</always_on>
-      <visualize>true</visualize>
-      <update_rate>30.0</update_rate>
-      <camera name="head">
-        <horizontal_fov>1.3962634</horizontal_fov>
-        <image>
-          <width>800</width>
-          <height>800</height>
-          <format>R8G8B8</format>
-        </image>
-        <clip>
-          <near>0.02</near>
-          <far>300</far>
-        </clip>
-        <noise>
-          <type>gaussian</type>
-          <!-- Noise is sampled independently per pixel on each frame.
-               That pixel's noise value is added to each of its color
-               channels, which at that point lie in the range [0,1]. -->
-          <mean>0.0</mean>
-          <stddev>0.007</stddev>
-        </noise>
-      </camera>
-      <plugin name="camera_controller" filename="libgazebo_ros_camera.so">
-        <alwaysOn>true</alwaysOn>
-        <robotNamespace>camera_bot</robotNamespace>
-        <updateRate>30.0</updateRate>
-        <cameraName>camera_bot/camera1</cameraName>
-        <imageTopicName>image_raw</imageTopicName>
-        <cameraInfoTopicName>camera_info</cameraInfoTopicName>
-        <frameName>camera_link</frameName>
-        <hackBaseline>0.07</hackBaseline>
-        <distortionK1>0.0</distortionK1>
-        <distortionK2>0.0</distortionK2>
-        <distortionK3>0.0</distortionK3>
-        <distortionT1>0.0</distortionT1>
-        <distortionT2>0.0</distortionT2>
-      </plugin>
+	<gazebo reference="camera_link">
+		<material>Gazebo/Red</material>
+		<sensor type="camera" name="camera">
+			<always_on>true</always_on>
+			<visualize>true</visualize>
+			<update_rate>30.0</update_rate>
+			<camera name="head">
+				<horizontal_fov>1.3962634</horizontal_fov>
+				<image>
+					<width>800</width>
+					<height>800</height>
+					<format>R8G8B8</format>
+				</image>
+				<clip>
+					<near>0.02</near>
+					<far>300</far>
+				</clip>
+				<noise>
+				<type>gaussian</type>
+					<!-- Noise is sampled independently per pixel on each frame.
+					That pixel's noise value is added to each of its color
+					channels, which at that point lie in the range [0,1]. -->
+					<mean>0.0</mean>
+					<stddev>0.007</stddev>
+				</noise>
+			</camera>
+			<plugin name="camera_controller" filename="libgazebo_ros_camera.so">
+				<alwaysOn>true</alwaysOn>
+				<robotNamespace>camera_bot</robotNamespace>
+				<updateRate>30.0</updateRate>
+				<cameraName>camera_bot/camera</cameraName>
+				<imageTopicName>image_raw</imageTopicName>
+				<cameraInfoTopicName>camera_info</cameraInfoTopicName>
+				<frameName>camera_link</frameName>
+				<hackBaseline>0.07</hackBaseline>
+				<distortionK1>0.0</distortionK1>
+				<distortionK2>0.0</distortionK2>
+				<distortionK3>0.0</distortionK3>
+				<distortionT1>0.0</distortionT1>
+				<distortionT2>0.0</distortionT2>
+			</plugin>
+		</sensor>
+    <sensor type="depth" name="depth_camera">
+		<always_on>true</always_on>
+		<visualize>true</visualize>
+		<update_rate>30.0</update_rate>
+		<topic>/depth_camera/depth_image</topic>
+		<camera name="head_depth">
+			<horizontal_fov>1.047198</horizontal_fov>
+			<image>
+				<width>640</width>
+				<height>480</height>
+				<format>R8G8B8</format>
+			</image>
+			<depth_camera></depth_camera>
+			<clip>
+				<near>0.05</near>
+				<far>3</far>
+			</clip>
+		</camera>
+        <plugin name="camera_plugin" filename="libgazebo_ros_openni_kinect.so">
+			<baseline>0.2</baseline>
+			<alwaysOn>true</alwaysOn>
+			<!-- Keep this zero, update_rate in the parent <sensor> tag
+			will control the frame rate. -->
+			<updateRate>0.0</updateRate>
+			<robotNamespace>camera_bot</robotNamespace>
+			<cameraName>depth_camera</cameraName>
+			<imageTopicName>image</imageTopicName>
+			<cameraInfoTopicName>camera_info</cameraInfoTopicName>
+			<depthImageTopicName>depth_image</depthImageTopicName>
+			<depthImageInfoTopicName>depth_camera_info</depthImageInfoTopicName>
+			<pointCloudTopicName>points</pointCloudTopicName>
+			<frameName>camera_link</frameName>
+			<pointCloudCutoff>0.05</pointCloudCutoff>
+			<distortionK1>0</distortionK1>
+			<distortionK2>0</distortionK2>
+			<distortionK3>0</distortionK3>
+			<distortionT1>0</distortionT1>
+			<distortionT2>0</distortionT2>
+			<CxPrime>0</CxPrime>
+			<Cx>0</Cx>
+			<Cy>0</Cy>
+			<focalLength>0</focalLength>
+			<hackBaseline>0</hackBaseline>
+        </plugin>
     </sensor>
   </gazebo>
